File: combo_low_profile_oled/dumbpad.kicad_pcb (KiCad board)
At the start: 2 copper layers, 97 x 78.5 mm, 43 parts, among them J1 Conn_01x04_Female

Commit message: - Updated README.md to reflect new revision 1.3.2 changes, including mounting points for uController cover and combined plated through holes for EC11 rotary encoder mounting points and sockets.
Parts:
- added MH1: MountingHole_2.1mm, MountingHole:MountingHole_2.1mm, F.Cu at (116.9, 111.0)
- added MH1: MountingHole_2.1mm, MountingHole:MountingHole_2.1mm, F.Cu at (104.2, 111.0)
Other:
- board text added: "dumbpad v1.3.2"
- board text removed: "dumbpad v1.3"
